File: pcb/DSKY_led_display.sch (KiCad schematic (older format))
At the start: 236 parts, among them J1 105133-0001, J2 20021221-00010C4LF, J3 TSM-104-01-L-SV, Q1 BSS138, Q2 BSS138, Q3 BSS138, Q4 BSS138, SW1 KMR241NG, U1 AP2204K-3.3, U2 LP5036, U3 LP5036, U4 LP5036, U5 LP5036, U6 ATSAMD21E18A-A, U7 LP5036, U8 LP5036

Commit message: validate pcb project is accessible from a second dev box
Parts:
- C1, C2, C3, C4, C6, C7, C8: Digi-Key_PN 399-C0603C105K3RAC7411CT-ND -> 399-C0603C105K3RAC7411CT-ND
- C5: Digi-Key_PN 311-3494-1-ND -> 311-3494-1-ND
- D10, D100, D101, D102, D103, D104, D105, D106, D107, D108, D109, D11, D110, D111, D112, D113, D114, D115, D116, D117, D118, D119, D12, D120, D121, D122, D123, D124, D125, D126, D127, D128, D129, D13, D130, D131, D132, D133, D134, D135, D136, D137, D138, D139, D14, D140, D141, D142, D143, D144, D145, D146, D147, D148, D149, D15, D150, D151, D152, D153, D154, D155, D156, D157, D158, D159, D16, D160, D161, D162, D163, D164, D165, D166, D167, D168, D169, D17, D170, D171, D172, D173, D174, D175, D176, D177, D178, D179, D18, D180, D181, D182, D183, D184, D185, D186, D187, D188, D189, D19, D190, D20, D21, D22, D23, D24, D25, D26, D27, D28, D29, D3, D30, D31, D32, D33, D34, D35, D36, D37, D38, D39, D4, D40, D41, D42, D43, D44, D45, D46, D47, D48, D49, D5, D50, D51, D52, D53, D54, D55, D56, D57, D58, D59, D6, D60, D61, D62, D63, D64, D65, D66, D67, D68, D69, D7, D70, D71, D72, D73, D74, D75, D76, D77, D78, D79, D8, D80, D81, D82, D83, D84, D85, D86, D87, D88, D89, D9, D90, D91, D92, D93, D94, D95, D96, D97, D98, D99: Digi-Key_PN 1830-1079-1-ND -> 1830-1079-1-ND
- J1: Digi-Key_PN WM9734CT-ND -> WM9734CT-ND
- J2: Digi-Key_PN 609-3700-1-ND -> 609-3700-1-ND
- R1, R2, R3, R6: Digi-Key_PN 541-4.7KGCT-ND -> 541-4.7KGCT-ND
- U1: Digi-Key_PN AP2204K-3.3TRG1DICT-ND -> AP2204K-3.3TRG1DICT-ND
- U2, U3, U4, U5, U7, U8: Digi-Key_PN 296-LP5036RJVRCT-ND -> 296-LP5036RJVRCT-ND

Commit message: V2 pcb as-ordered for testing
Parts:
- added C10, C11, C12, C13, C14, C9: 1 uF, Capacitor_SMD:C_0603_1608Metric, symbol Device:C_Small
- C1, C2, C3, C4, C6, C7, C8: Digi-Key_PN 399-C0603C105K3RAC7411CT-ND -> 399-C0603C105K3RAC7411CT-ND
- C5: Digi-Key_PN 311-3494-1-ND -> 311-3494-1-ND
- D10, D100, D101, D102, D103, D104, D105, D106, D107, D108, D109, D11, D110, D111, D112, D113, D114, D115, D116, D117, D118, D119, D12, D120, D121, D122, D123, D124, D125, D126, D127, D128, D129, D13, D130, D131, D132, D133, D134, D135, D136, D137, D138, D139, D14, D140, D141, D142, D143, D144, D145, D146, D147, D148, D149, D15, D150, D151, D152, D153, D154, D155, D156, D157, D158, D159, D16, D160, D161, D162, D163, D164, D165, D166, D167, D168, D169, D17, D170, D171, D172, D173, D174, D175, D176, D177, D178, D179, D18, D180, D181, D182, D183, D184, D185, D186, D187, D188, D189, D19, D190, D20, D21, D22, D23, D24, D25, D26, D27, D28, D29, D3, D30, D31, D32, D33, D34, D35, D36, D37, D38, D39, D4, D40, D41, D42, D43, D44, D45, D46, D47, D48, D49, D5, D50, D51, D52, D53, D54, D55, D56, D57, D58, D59, D6, D60, D61, D62, D63, D64, D65, D66, D67, D68, D69, D7, D70, D71, D72, D73, D74, D75, D76, D77, D78, D79, D8, D80, D81, D82, D83, D84, D85, D86, D87, D88, D89, D9, D90, D91, D92, D93, D94, D95, D96, D97, D98, D99: Digi-Key_PN 1830-1079-1-ND -> 1830-1079-1-ND
- J1: Digi-Key_PN WM9734CT-ND -> WM9734CT-ND
- J2: Digi-Key_PN 609-3700-1-ND -> 609-3700-1-ND
- R1, R2, R3, R6: Digi-Key_PN 541-4.7KGCT-ND -> 541-4.7KGCT-ND
- U1: Digi-Key_PN AP2204K-3.3TRG1DICT-ND -> AP2204K-3.3TRG1DICT-ND
- U2, U3, U4, U5, U7, U8: Digi-Key_PN 296-LP5036RJVRCT-ND -> 296-LP5036RJVRCT-ND
Connections:
- net +5V: no longer U2.45 (VCAP), U3.45 (VCAP), U4.45 (VCAP), U5.45 (VCAP), U7.45 (VCAP), U8.45 (VCAP)
- net GND: now also C10.2, C11.2, C12.2, C13.2, C14.2, C9.2
- new net: C9.1, U2.45 (VCAP)
- new net: C11.1, U5.45 (VCAP)
- new net: C14.1, U8.45 (VCAP)
- new net: C13.1, U7.45 (VCAP)
- new net: C12.1, U4.45 (VCAP)
- new net: C10.1, U3.45 (VCAP)

Commit message: V3 board
Parts:
- removed Q1, Q2, Q3, Q4: BSS138, digikey-footprints:SOT-23-3, symbol dk_Transistors-FETs-MOSFETs-Single:BSS138
- removed R13, R14: 10K, Resistor_SMD:R_0603_1608Metric, symbol Device:R
- added C15: 10 uF, Capacitor_SMD:C_0603_1608Metric, symbol Device:C_Small
- added U9: TCA9543ADR, Package_SO:SOIC-14_3.9x8.7mm_P1.27mm, symbol project-symbols:TCA9543ADR
- J2: value 20021221-00010C4LF -> 3221-10-0300-00-TR; Digi-Key_PN 609-3700-1-ND -> 1175-2649-1-ND
- R10, R8, R9: value 10K -> 1K; Description RES SMD 10K OHM 5% 1/10W 0603 -> RES SMD 1K OHM 5% 1/10W 0603; Digi-Key_PN 541-1804-1-ND -> 541-4.7KGCT-ND
- R11, R12: value 10K -> 4.7K; Description RES SMD 10K OHM 5% 1/10W 0603 -> RES SMD 4.7K OHM 5% 1/10W 0603; Digi-Key_PN 541-1804-1-ND -> 541-4.7KGCT-ND
- R7: value 10K -> 1K; Description RES SMD 10K OHM 5% 1/10W 0603 -> RES SMD 4.7K OHM 5% 1/10W 0603; Digi-Key_PN 541-1804-1-ND -> 541-4.7KGCT-ND
Connections:
- net +3V3: now also C15.1, U9.14 (VCC); no longer R11.2, R7.2, R9.2
- net 3SCL: now also U9.13 (SDA)
- net 3SDA: now also U9.12 (SCL); no longer R11.1
- net D+: now also U6.24 (PA25); no longer U6.23 (PA24)
- net D-: now also U6.23 (PA24); no longer U6.22 (PA23)
- net GND: now also C15.2, U9.1 (A0), U9.2 (A1), U9.7 (GND)
- net BRESET: now reaches U6.3 (PA02)
- net BRESET: now also U9.3 (RESET)
- net at R2.2, U5.38 (ADDR0), U5.39 (ADDR1): now also U5.43 (EN)
- net at R6.2, U7.38 (ADDR0): now also U7.43 (EN)
- net at R1.2, U4.38 (ADDR0): now also U4.43 (EN)
- net at R3.2, U3.39 (ADDR1): now also U3.43 (EN)
- net +5V renamed VCC
- net VCC: now also R10.1, R11.1, R12.1, R7.1, R8.1, R9.1; no longer R10.2, R12.2, R8.2
- net 3EN0: no longer names the net of U6.1 (PA00)
- net 3EN0: no longer R7.1
- net 3EN1: no longer names the net of U6.2 (PA01)
- net 3EN1: no longer R9.1
- removed net EN0: R8.1, U2.43 (EN), U3.43 (EN), U4.43 (EN), U5.43 (EN)
- removed net EN1: R10.1, U7.43 (EN), U8.43 (EN)
- net SCL renamed SCL0
- net SCL0: now also R7.2, U9.6 (SCL0); no longer U7.42 (SCL), U8.42 (SCL)
- net SDA renamed SDA0
- net SDA0: now also R8.2, U9.5 (SDA0); no longer R12.1, U7.41 (SDA), U8.41 (SDA)
- new net: R11.2, U2.43 (EN)
- new net: R12.2, U8.43 (EN)
- new net SCL1: R9.2, U7.42 (SCL), U8.42 (SCL), U9.10 (SCL1)
- new net SDA1: R10.2, U7.41 (SDA), U8.41 (SDA), U9.9 (SDA1)
- no-connect marks 59 -> 57
Other:
- note added: "I2C Bus 0"
- note added: "I2C Bus 1"
- note added: "Main I2C Bus"
- note removed: "3.3V \nI2C++ BUS"
- note removed: "5V \nI2C++ BUS"
- moved on the sheet: SW1

Commit message: V4 board
Version 4 of the PCB
Parts:
- removed R1, R11, R12, R2, R3, R6: 4.7K, Resistor_SMD:R_0603_1608Metric, symbol Device:R
- added R13: 0K, Resistor_SMD:R_0603_1608Metric, symbol Device:R
- added R14, R21, R22, R23: 1K, Resistor_SMD:R_0603_1608Metric, symbol Device:R
Connections:
- net +3V3: now also R13.1, R14.1, R21.1
- net 3SCL: now also U9.12 (SCL), R21.2; no longer U9.13 (SDA)
- net 3SDA: now also U9.13 (SDA), R14.2; no longer U9.12 (SCL)
- net BRESET: now also U6.1 (PA00), R13.2; no longer U6.3 (PA02)
- net GND: no longer D10.1 (K), D100.1 (K), D101.1 (K), D102.1 (K), D103.1 (K), D104.1 (K), D105.1 (K), D106.1 (K), D107.1 (K), D108.1 (K), D109.1 (K), D11.1 (K), D110.1 (K), D111.1 (K), D112.1 (K), D113.1 (K), D114.1 (K), D115.1 (K), D116.1 (K), D117.1 (K), D118.1 (K), D119.1 (K), D12.1 (K), D120.1 (K), D121.1 (K), D122.1 (K), D123.1 (K), D124.1 (K), D125.1 (K), D126.1 (K), D127.1 (K), D128.1 (K), D129.1 (K), D13.1 (K), D130.1 (K), D131.1 (K), D132.1 (K), D133.1 (K), D134.1 (K), D135.1 (K), D136.1 (K), D137.1 (K), D138.1 (K), D139.1 (K), D14.1 (K), D140.1 (K), D141.1 (K), D142.1 (K), D143.1 (K), D144.1 (K), D145.1 (K), D146.1 (K), D147.1 (K), D148.1 (K), D149.1 (K), D15.1 (K), D150.1 (K), D151.1 (K), D152.1 (K), D153.1 (K), D154.1 (K), D155.1 (K), D156.1 (K), D157.1 (K), D158.1 (K), D159.1 (K), D16.1 (K), D160.1 (K), D161.1 (K), D162.1 (K), D163.1 (K), D164.1 (K), D165.1 (K), D166.1 (K), D167.1 (K), D168.1 (K), D169.1 (K), D17.1 (K), D170.1 (K), D171.1 (K), D172.1 (K), D173.1 (K), D174.1 (K), D175.1 (K), D176.1 (K), D177.1 (K), D178.1 (K), D179.1 (K), D18.1 (K), D180.1 (K), D181.1 (K), D182.1 (K), D183.1 (K), D184.1 (K), D185.1 (K), D186.1 (K), D187.1 (K), D188.1 (K), D189.1 (K), D19.1 (K), D190.1 (K), D20.1 (K), D21.1 (K), D22.1 (K), D23.1 (K), D24.1 (K), D25.1 (K), D26.1 (K), D27.1 (K), D28.1 (K), D29.1 (K), D3.1 (K), D30.1 (K), D31.1 (K), D32.1 (K), D33.1 (K), D34.1 (K), D35.1 (K), D36.1 (K), D37.1 (K), D38.1 (K), D39.1 (K), D4.1 (K), D40.1 (K), D41.1 (K), D42.1 (K), D43.1 (K), D44.1 (K), D45.1 (K), D46.1 (K), D47.1 (K), D48.1 (K), D49.1 (K), D5.1 (K), D50.1 (K), D51.1 (K), D52.1 (K), D53.1 (K), D54.1 (K), D55.1 (K), D56.1 (K), D57.1 (K), D58.1 (K), D59.1 (K), D6.1 (K), D60.1 (K), D61.1 (K), D62.1 (K), D63.1 (K), D64.1 (K), D65.1 (K), D66.1 (K), D67.1 (K), D68.1 (K), D69.1 (K), D7.1 (K), D70.1 (K), D71.1 (K), D72.1 (K), D73.1 (K), D74.1 (K), D75.1 (K), D76.1 (K), D77.1 (K), D78.1 (K), D79.1 (K), D8.1 (K), D80.1 (K), D81.1 (K), D82.1 (K), D83.1 (K), D84.1 (K), D85.1 (K), D86.1 (K), D87.1 (K), D88.1 (K), D89.1 (K), D9.1 (K), D90.1 (K), D91.1 (K), D92.1 (K), D93.1 (K), D94.1 (K), D95.1 (K), D96.1 (K), D97.1 (K), D98.1 (K), D99.1 (K)
- net VCC: now also D10.2 (A), D100.2 (A), D101.2 (A), D102.2 (A), D103.2 (A), D104.2 (A), D105.2 (A), D106.2 (A), D107.2 (A), D108.2 (A), D109.2 (A), D11.2 (A), D110.2 (A), D111.2 (A), D112.2 (A), D113.2 (A), D114.2 (A), D115.2 (A), D116.2 (A), D117.2 (A), D118.2 (A), D119.2 (A), D12.2 (A), D120.2 (A), D121.2 (A), D122.2 (A), D123.2 (A), D124.2 (A), D125.2 (A), D126.2 (A), D127.2 (A), D128.2 (A), D129.2 (A), D13.2 (A), D130.2 (A), D131.2 (A), D132.2 (A), D133.2 (A), D134.2 (A), D135.2 (A), D136.2 (A), D137.2 (A), D138.2 (A), D139.2 (A), D14.2 (A), D140.2 (A), D141.2 (A), D142.2 (A), D143.2 (A), D144.2 (A), D145.2 (A), D146.2 (A), D147.2 (A), D148.2 (A), D149.2 (A), D15.2 (A), D150.2 (A), D151.2 (A), D152.2 (A), D153.2 (A), D154.2 (A), D155.2 (A), D156.2 (A), D157.2 (A), D158.2 (A), D159.2 (A), D16.2 (A), D160.2 (A), D161.2 (A), D162.2 (A), D163.2 (A), D164.2 (A), D165.2 (A), D166.2 (A), D167.2 (A), D168.2 (A), D169.2 (A), D17.2 (A), D170.2 (A), D171.2 (A), D172.2 (A), D173.2 (A), D174.2 (A), D175.2 (A), D176.2 (A), D177.2 (A), D178.2 (A), D179.2 (A), D18.2 (A), D180.2 (A), D181.2 (A), D182.2 (A), D183.2 (A), D184.2 (A), D185.2 (A), D186.2 (A), D187.2 (A), D188.2 (A), D189.2 (A), D19.2 (A), D190.2 (A), D20.2 (A), D21.2 (A), D22.2 (A), D23.2 (A), D24.2 (A), D25.2 (A), D26.2 (A), D27.2 (A), D28.2 (A), D29.2 (A), D3.2 (A), D30.2 (A), D31.2 (A), D32.2 (A), D33.2 (A), D34.2 (A), D35.2 (A), D36.2 (A), D37.2 (A), D38.2 (A), D39.2 (A), D4.2 (A), D40.2 (A), D41.2 (A), D42.2 (A), D43.2 (A), D44.2 (A), D45.2 (A), D46.2 (A), D47.2 (A), D48.2 (A), D49.2 (A), D5.2 (A), D50.2 (A), D51.2 (A), D52.2 (A), D53.2 (A), D54.2 (A), D55.2 (A), D56.1 (K), D57.2 (A), D58.2 (A), D59.2 (A), D6.2 (A), D60.2 (A), D61.2 (A), D62.2 (A), D63.2 (A), D64.2 (A), D65.2 (A), D66.2 (A), D67.2 (A), D68.2 (A), D69.2 (A), D7.2 (A), D70.2 (A), D71.2 (A), D72.2 (A), D73.2 (A), D74.2 (A), D75.2 (A), D76.2 (A), D77.2 (A), D78.2 (A), D79.2 (A), D8.2 (A), D80.2 (A), D81.2 (A), D82.2 (A), D83.2 (A), D84.2 (A), D85.2 (A), D86.2 (A), D87.2 (A), D88.2 (A), D89.2 (A), D9.2 (A), D90.2 (A), D91.2 (A), D92.2 (A), D93.2 (A), D94.2 (A), D95.2 (A), D96.2 (A), D97.2 (A), D98.2 (A), D99.2 (A), U2.43 (EN), U3.39 (ADDR1), U3.43 (EN), U4.38 (ADDR0), U4.43 (EN), U5.38 (ADDR0), U5.39 (ADDR1), U5.43 (EN), U7.38 (ADDR0), U7.43 (EN), U8.43 (EN), R22.1, R23.1
- net abus0: now also D69.1 (K); no longer D69.2 (A)
- net abus1: now also D76.1 (K); no longer D76.2 (A)
- net abus10: now also D103.1 (K); no longer D103.2 (A)
- net abus11: now also D95.1 (K); no longer D95.2 (A)
- net abus12: now also D77.1 (K); no longer D77.2 (A)
- net abus13: now also D87.1 (K); no longer D87.2 (A)
- net abus14: now also D71.1 (K); no longer D71.2 (A)
- net abus15: now also D80.1 (K); no longer D80.2 (A)
- net abus16: now also D94.1 (K); no longer D94.2 (A)
- net abus17: now also D104.1 (K); no longer D104.2 (A)
- net abus18: now also D96.1 (K); no longer D96.2 (A)
- net abus19: now also D78.1 (K); no longer D78.2 (A)
- net abus2: now also D91.1 (K); no longer D91.2 (A)
- net abus20: now also D88.1 (K); no longer D88.2 (A)
- net abus21: now also D72.1 (K); no longer D72.2 (A)
- net abus22: now also D83.1 (K); no longer D83.2 (A)
- net abus23: now also D97.1 (K); no longer D97.2 (A)
- net abus24: now also D105.1 (K); no longer D105.2 (A)
- net abus25: now also D99.1 (K); no longer D99.2 (A)
- net abus26: now also D81.1 (K); no longer D81.2 (A)
- net abus27: now also D89.1 (K); no longer D89.2 (A)
- net abus28: now also D73.1 (K); no longer D73.2 (A)
- net abus29: now also D84.1 (K); no longer D84.2 (A)
- net abus3: now also D101.1 (K); no longer D101.2 (A)
- net abus30: now also D98.1 (K); no longer D98.2 (A)
- net abus31: now also D106.1 (K); no longer D106.2 (A)
- net abus32: now also D100.1 (K); no longer D100.2 (A)
- net abus33: now also D82.1 (K); no longer D82.2 (A)
- net abus34: now also D90.1 (K); no longer D90.2 (A)
- net abus4: now also D92.1 (K); no longer D92.2 (A)
- net abus5: now also D75.1 (K); no longer D75.2 (A)
- net abus6: now also D85.1 (K); no longer D85.2 (A)
- net abus7: now also D70.1 (K); no longer D70.2 (A)
- net abus8: now also D79.1 (K); no longer D79.2 (A)
- net abus9: now also D93.1 (K); no longer D93.2 (A)
- net bbus0: now also D111.1 (K); no longer D111.2 (A)
- net bbus1: now also D118.1 (K); no longer D118.2 (A)
- net bbus10: now also D145.1 (K); no longer D145.2 (A)
- net bbus11: now also D137.1 (K); no longer D137.2 (A)
- net bbus12: now also D119.1 (K); no longer D119.2 (A)
- net bbus13: now also D129.1 (K); no longer D129.2 (A)
- net bbus14: now also D114.1 (K); no longer D114.2 (A)
- net bbus15: now also D122.1 (K); no longer D122.2 (A)
- net bbus16: now also D136.1 (K); no longer D136.2 (A)
- net bbus17: now also D146.1 (K); no longer D146.2 (A)
- net bbus18: now also D138.1 (K); no longer D138.2 (A)
- net bbus19: now also D120.1 (K); no longer D120.2 (A)
- net bbus2: now also D133.1 (K); no longer D133.2 (A)
- net bbus20: now also D130.1 (K); no longer D130.2 (A)
- net bbus21: now also D115.1 (K); no longer D115.2 (A)
- net bbus22: now also D125.1 (K); no longer D125.2 (A)
- net bbus23: now also D139.1 (K); no longer D139.2 (A)
- net bbus24: now also D147.1 (K); no longer D147.2 (A)
- net bbus25: now also D141.1 (K); no longer D141.2 (A)
- net bbus26: now also D123.1 (K); no longer D123.2 (A)
- net bbus27: now also D131.1 (K); no longer D131.2 (A)
- net bbus28: now also D116.1 (K); no longer D116.2 (A)
- net bbus29: now also D126.1 (K); no longer D126.2 (A)
- net bbus3: now also D144.1 (K); no longer D144.2 (A)
- net bbus30: now also D140.1 (K); no longer D140.2 (A)
- net bbus31: now also D148.1 (K); no longer D148.2 (A)
- net bbus32: now also D142.1 (K); no longer D142.2 (A)
- net bbus33: now also D124.1 (K); no longer D124.2 (A)
- net bbus34: now also D132.1 (K); no longer D132.2 (A)
- net bbus4: now also D134.1 (K); no longer D134.2 (A)
- net bbus5: now also D117.1 (K); no longer D117.2 (A)
- net bbus6: now also D128.1 (K); no longer D128.2 (A)
- net bbus7: now also D113.1 (K); no longer D113.2 (A)
- net bbus8: now also D121.1 (K); no longer D121.2 (A)
- net bbus9: now also D135.1 (K); no longer D135.2 (A)
- net cbus0: now also D154.1 (K); no longer D154.2 (A)
- net cbus1: now also D160.1 (K); no longer D160.2 (A)
- net cbus10: now also D187.1 (K); no longer D187.2 (A)
- net cbus11: now also D180.1 (K); no longer D180.2 (A)
- net cbus12: now also D161.1 (K); no longer D161.2 (A)
- net cbus13: now also D171.1 (K); no longer D171.2 (A)
- net cbus14: now also D156.1 (K); no longer D156.2 (A)
- net cbus15: now also D165.1 (K); no longer D165.2 (A)
- net cbus16: now also D179.1 (K); no longer D179.2 (A)
- net cbus17: now also D188.1 (K); no longer D188.2 (A)
- net cbus18: now also D181.1 (K); no longer D181.2 (A)
- net cbus19: now also D162.1 (K); no longer D162.2 (A)
- net cbus2: now also D175.1 (K); no longer D175.2 (A)
- net cbus20: now also D172.1 (K); no longer D172.2 (A)
- net cbus21: now also D157.1 (K); no longer D157.2 (A)
- net cbus22: now also D168.1 (K); no longer D168.2 (A)
- net cbus23: now also D182.1 (K); no longer D182.2 (A)
- net cbus24: now also D189.1 (K); no longer D189.2 (A)
- net cbus25: now also D184.1 (K); no longer D184.2 (A)
- net cbus26: now also D166.1 (K); no longer D166.2 (A)
- net cbus27: now also D173.1 (K); no longer D173.2 (A)
- net cbus28: now also D158.1 (K); no longer D158.2 (A)
- net cbus29: now also D169.1 (K); no longer D169.2 (A)
- net cbus3: now also D186.1 (K); no longer D186.2 (A)
- net cbus30: now also D183.1 (K); no longer D183.2 (A)
- net cbus31: now also D190.1 (K); no longer D190.2 (A)
- net cbus32: now also D185.1 (K); no longer D185.2 (A)
- net cbus33: now also D167.1 (K); no longer D167.2 (A)
- net cbus34: now also D174.1 (K); no longer D174.2 (A)
- net cbus4: now also D177.1 (K); no longer D177.2 (A)
- net cbus5: now also D159.1 (K); no longer D159.2 (A)
- net cbus6: now also D170.1 (K); no longer D170.2 (A)
- net cbus7: now also D155.1 (K); no longer D155.2 (A)
- net cbus8: now also D164.1 (K); no longer D164.2 (A)
- net cbus9: now also D178.1 (K); no longer D178.2 (A)
- net dbus0: now also D15.1 (K); no longer D15.2 (A)
- net dbus1: now also D19.1 (K); no longer D19.2 (A)
- net dbus10: now also D28.1 (K); no longer D28.2 (A)
- net dbus11: now also D26.1 (K); no longer D26.2 (A)
- net dbus12: now also D18.1 (K); no longer D18.2 (A)
- net dbus13: now also D22.1 (K); no longer D22.2 (A)
- net dbus2: now also D23.1 (K); no longer D23.2 (A)
- net dbus3: now also D27.1 (K); no longer D27.2 (A)
- net dbus4: now also D25.1 (K); no longer D25.2 (A)
- net dbus5: now also D17.1 (K); no longer D17.2 (A)
- net dbus6: now also D21.1 (K); no longer D21.2 (A)
- net dbus7: now also D16.1 (K); no longer D16.2 (A)
- net dbus8: now also D20.1 (K); no longer D20.2 (A)
- net dbus9: now also D24.1 (K); no longer D24.2 (A)
- net ebus0: now also D37.1 (K); no longer D37.2 (A)
- net ebus1: now also D43.1 (K); no longer D43.2 (A)
- net ebus10: now also D62.1 (K); no longer D62.2 (A)
- net ebus12: now also D42.1 (K); no longer D42.2 (A)
- net ebus13: now also D50.1 (K); no longer D50.2 (A)
- net ebus2: now also D53.1 (K); no longer D53.2 (A)
- net ebus3: now also D61.1 (K); no longer D61.2 (A)
- net ebus4: now also D55.1 (K); no longer D55.2 (A)
- net ebus5: now also D41.1 (K); no longer D41.2 (A)
- net ebus6: now also D49.1 (K); no longer D49.2 (A)
- net ebus7: now also D38.1 (K); no longer D38.2 (A)
- net ebus8: now also D44.1 (K); no longer D44.2 (A)
- net ebus9: now also D54.1 (K); no longer D54.2 (A)
- net fbus0: now also D39.1 (K); no longer D39.2 (A)
- net fbus1: now also D47.1 (K); no longer D47.2 (A)
- net fbus10: now also D64.1 (K); no longer D64.2 (A)
- net fbus11: now also D60.1 (K); no longer D60.2 (A)
- net fbus12: now also D46.1 (K); no longer D46.2 (A)
- net fbus13: now also D52.1 (K); no longer D52.2 (A)
- net fbus2: now also D57.1 (K); no longer D57.2 (A)
- net fbus3: now also D63.1 (K); no longer D63.2 (A)
- net fbus4: now also D59.1 (K); no longer D59.2 (A)
- net fbus5: now also D45.1 (K); no longer D45.2 (A)
- net fbus6: now also D51.1 (K); no longer D51.2 (A)
- net fbus7: now also D40.1 (K); no longer D40.2 (A)
- net fbus8: now also D48.1 (K); no longer D48.2 (A)
- net fbus9: now also D58.1 (K); no longer D58.2 (A)
- net g0bus0: now also D3.1 (K); no longer D3.2 (A)
- net g0bus1: now also D10.1 (K); no longer D10.2 (A)
- net g0bus2: now also D4.1 (K); no longer D4.2 (A)
- net g0bus3: now also D7.1 (K); no longer D7.2 (A)
- net g0bus4: now also D13.1 (K); no longer D13.2 (A)
- net g0bus5: now also D12.1 (K); no longer D12.2 (A)
- net g0bus6: now also D11.1 (K); no longer D11.2 (A)
- net g0bus7: now also D14.1 (K); no longer D14.2 (A)
- net g1bus0: now also D5.1 (K); no longer D5.2 (A)
- net g1bus1: now also D8.1 (K); no longer D8.2 (A)
- net g1bus2: now also D9.1 (K); no longer D9.2 (A)
- net g1bus3: now also D6.1 (K); no longer D6.2 (A)
- net g2bus0: now also D29.1 (K); no longer D29.2 (A)
- net g2bus1: now also D33.1 (K); no longer D33.2 (A)
- net g2bus2: now also D34.1 (K); no longer D34.2 (A)
- net g2bus3: now also D30.1 (K); no longer D30.2 (A)
- net g3bus0: now also D31.1 (K); no longer D31.2 (A)
- net g3bus1: now also D35.1 (K); no longer D35.2 (A)
- net g3bus2: now also D36.1 (K); no longer D36.2 (A)
- net g3bus3: now also D32.1 (K); no longer D32.2 (A)
- net g4bus0: now also D65.1 (K); no longer D65.2 (A)
- net g4bus1: now also D66.1 (K); no longer D66.2 (A)
- net g4bus2: now also D67.1 (K); no longer D67.2 (A)
- net g4bus3: now also D68.1 (K); no longer D68.2 (A)
- net g5bus0: now also D107.1 (K); no longer D107.2 (A)
- net g5bus1: now also D108.1 (K); no longer D108.2 (A)
- net g5bus2: now also D109.1 (K); no longer D109.2 (A)
- net g5bus3: now also D110.1 (K); no longer D110.2 (A)
- net g6bus0: now also D149.1 (K); no longer D149.2 (A)
- net g6bus1: now also D150.1 (K); no longer D150.2 (A)
- net g6bus2: now also D151.1 (K); no longer D151.2 (A)
- net g6bus3: now also D152.1 (K); no longer D152.2 (A)
- net sabus0: now also D74.1 (K); no longer D74.2 (A)
- net sabus1: now also D86.1 (K); no longer D86.2 (A)
- net sabus2: now also D102.1 (K); no longer D102.2 (A)
- net sbbus0: now also D112.1 (K); no longer D112.2 (A)
- net sbbus1: now also D127.1 (K); no longer D127.2 (A)
- net sbbus2: now also D143.1 (K); no longer D143.2 (A)
- net scbus0: now also D153.1 (K); no longer D153.2 (A)
- net scbus1: now also D163.1 (K); no longer D163.2 (A)
- net scbus2: now also D176.1 (K); no longer D176.2 (A)
- net at U9.4 (INT0): now also R22.2
- net at U9.8 (INT1): now also R23.2
- no-connect marks 57 -> 55
Other:
- note added: "DNP"
- moved on the sheet: C5, D1, D10, D100, D101, D102, D103, D104, D105, D106, D107, D108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
