File: pcb/DSKY_led_display.kicad_pcb (KiCad board)
At the start: 4 copper layers, 63.5 x 105.5 mm, 238 parts, among them J1 105133-0001, J2 3221-10-0300-00-TR, J3 TSM-104-01-L-SV, SW1 KMR241NG, U1 AP2204K-3.3, U2 LP5036, U3 LP5036, U4 LP5036, U5 LP5036, U6 ATSAMD21E18A-A, U7 LP5036, U8 LP5036, U9 TCA9543ADR

Commit message: Update owing to KiCad V7 being fussier about bus definitions
Connections:
- net /sabus0 renamed sabus0
- net /sabus1 renamed sabus1
- net /sabus2 renamed sabus2
- net /sbbus0 renamed sbbus0
- net /sbbus1 renamed sbbus1
- net /sbbus2 renamed sbbus2
- net /scbus0 renamed scbus0
- net /scbus1 renamed scbus1
- net /scbus2 renamed scbus2
Changed lines of the file:
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@@
       (drillshape 0)
       (scaleselection 1)
-      (outputdirectory "gerber-V6/")
+      (outputdirectory "gerber-V7/")
     )
   )
@@
   (net 156 "g6bus2")
   (net 157 "g6bus3")
-  (net 158 "/sabus0")
+  (net 158 "sabus0")
   (net 159 "cbus0")
   (net 160 "cbus7")
@@
   (net 166 "cbus12")
   (net 167 "cbus19")
-  (net 168 "/sabus1")
+  (net 168 "sabus1")
   (net 169 "cbus8")
   (net 170 "cbus15")
@@
   (net 179 "cbus34")
   (net 180 "cbus2")
-  (net 181 "/sabus2")
+  (net 181 "sabus2")
   (net 182 "cbus4")
   (net 183 "cbus9")
@@
   (net 196 "/3SDA")
   (net 197 "/3SCL")
-  (net 198 "/sbbus0")
-  (net 199 "/sbbus1")
-  (net 200 "/sbbus2")
-  (net 201 "/scbus0")
-  (net 202 "/scbus1")
-  (net 203 "/scbus2")
+  (net 198 "sbbus0")
+  (net 199 "sbbus1")
+  (net 200 "sbbus2")
+  (net 201 "scbus0")
+  (net 202 "scbus1")
+  (net 203 "scbus2")
   (net 204 "Net-(D191-K)")
   (net 205 "/SWCLK")
@@
       (net 37 "g3bus3") (pinfunction "OUT25") (pintype "power_out"))
     (pad "27" smd roundrect (at 2.4625 1.2) (size 0.825 0.2) (layers "F.Cu" "F.Paste" "F.Mask") (roundrect_rratio 0.25)
-      (net 158 "/sabus0") (pinfunction "OUT26") (pintype "power_out"))
+      (net 158 "sabus0") (pinfunction "OUT26") (pintype "power_out"))
     (pad "28" smd roundrect (at 2.4625 0.8) (size 0.825 0.2) (layers "F.Cu" "F.Paste" "F.Mask") (roundrect_rratio 0.25)
-      (net 168 "/sabus1") (pinfunction "OUT27") (pintype "power_out"))
+      (net 168 "sabus1") (pinfunction "OUT27") (pintype "power_out"))
     (pad "29" smd roundrect (at 2.4625 0.4) (size 0.825 0.2) (layers "F.Cu" "F.Paste" "F.Mask") (roundrect_rratio 0.25)
-      (net 181 "/sabus2") (pinfunction "OUT28") (pintype "power_out"))
+      (net 181 "sabus2") (pinfunction "OUT28") (pintype "power_out"))
     (pad "30" smd roundrect (at 2.4625 0) (size 0.825 0.2) (layers "F.Cu" "F.Paste" "F.Mask") (roundrect_rratio 0.25)
-      (net 198 "/sbbus0") (pinfunction "OUT29") (pintype "power_out"))
+      (net 198 "sbbus0") (pinfunction "OUT29") (pintype "power_out"))
     (pad "31" smd roundrect (at 2.4625 -0.4) (size 0.825 0.2) (layers "F.Cu" "F.Paste" "F.Mask") (roundrect_rratio 0.25)
-      (net 199 "/sbbus1") (pinfunction "OUT30") (pintype "power_out"))
+      (net 199 "sbbus1") (pinfunction "OUT30") (pintype "power_out"))
     (pad "32" smd roundrect (at 2.4625 -0.8) (size 0.825 0.2) (layers "F.Cu" "F.Paste" "F.Mask") (roundrect_rratio 0.25)
-      (net 200 "/sbbus2") (pinfunction "OUT31") (pintype "power_out"))
+      (net 200 "sbbus2") (pinfunction "OUT31") (pintype "power_out"))
     (pad "33" smd roundrect (at 2.4625 -1.2) (size 0.825 0.2) (layers "F.Cu" "F.Paste" "F.Mask") (roundrect_rratio 0.25)
-      (net 201 "/scbus0") (pinfunction "OUT32") (pintype "power_out"))
+      (net 201 "scbus0") (pinfunction "OUT32") (pintype "power_out"))
     (pad "34" smd roundrect (at 2.4625 -1.6) (size 0.825 0.2) (layers "F.Cu" "F.Paste" "F.Mask") (roundrect_rratio 0.25)
-      (net 202 "/scbus1") (pinfunction "OUT33") (pintype "power_out"))
+      (net 202 "scbus1") (pinfunction "OUT33") (pintype "power_out"))
     (pad "35" smd roundrect (at 2.4625 -2) (size 0.825 0.2) (layers "F.Cu" "F.Paste" "F.Mask") (roundrect_rratio 0.25)
-      (net 203 "/scbus2") (pinfunction "OUT34") (pintype "power_out"))
+      (net 203 "scbus2") (pinfunction "OUT34") (pintype "power_out"))
     (pad "36" smd roundrect (at 2.4625 -2.4) (size 0.825 0.2) (layers "F.Cu" "F.Paste" "F.Mask") (roundrect_rratio 0.25)
       (net 278 "unconnected-(U8-OUT35-Pad36)") (pinfunction "OUT35") (pintype "power_out+no_connect"))
@@
       (stroke (width 0.1) (type solid)) (layer "B.Fab"))
     (pad "1" smd roundrect (at -0.9375 0 90) (size 0.975 1.4) (layers "B.Cu" "B.Paste" "B.Mask") (roundrect_rratio 0.25)
-      (net 158 "/sabus0") (pinfunction "K") (pintype "passive"))
+      (net 158 "sabus0") (pinfunction "K") (pintype "passive"))
     (pad "2" smd roundrect (at 0.9375 0 90) (size 0.975 1.4) (layers "B.Cu" "B.Paste" "B.Mask") (roundrect_rratio 0.25)
       (net 221 "VCC") (pinfunction "A") (pintype "passive"))
@@
       (stroke (width 0.1) (type solid)) (layer "B.Fab"))
     (pad "1" smd roundrect (at -0.9375 0) (size 0.975 1.4) (layers "B.Cu" "B.Paste" "B.Mask") (roundrect_rratio 0.25)
-      (net 168 "/sabus1") (pinfunction "K") (pintype "passive"))
+      (net 168 "sabus1") (pinfunction "K") (pintype "passive"))
     (pad "2" smd roundrect (at 0.9375 0) (size 0.975 1.4) (layers "B.Cu" "B.Paste" "B.Mask") (roundrect_rratio 0.25)
       (net 221 "VCC") (pinfunction "A") (pintype "passive"))
@@
       (stroke (width 0.1) (type solid)) (layer "B.Fab"))
     (pad "1" smd roundrect (at -0.9375 0 90) (size 0.975 1.4) (layers "B.Cu" "B.Paste" "B.Mask") (roundrect_rratio 0.25)
-      (net 181 "/sabus2") (pinfunction "K") (pintype "passive"))
+      (net 181 "sabus2") (pinfunction "K") (pintype "passive"))
     (pad "2" smd roundrect (at 0.9375 0 90) (size 0.975 1.4) (layers "B.Cu" "B.Paste" "B.Mask") (roundrect_rratio 0.25)
       (net 221 "VCC") (pinfunction "A") (pintype "passive"))
@@
       (stroke (width 0.1) (type solid)) (layer "B.Fab"))
     (pad "1" smd roundrect (at -0.9375 0 90) (size 0.975 1.4) (layers "B.Cu" "B.Paste" "B.Mask") (roundrect_rratio 0.25)
-      (net 198 "/sbbus0") (pinfunction "K") (pintype "passive"))
+      (net 198 "sbbus0") (pinfunction "K") (pintype "passive"))
     (pad "2" smd roundrect (at 0.9375 0 90) (size 0.975 1.4) (layers "B.Cu" "B.Paste" "B.Mask") (roundrect_rratio 0.25)
       (net 221 "VCC") (pinfunction "A") (pintype "passive"))
@@
       (stroke (width 0.1) (type solid)) (layer "B.Fab"))
     (pad "1" smd roundrect (at -0.9375 0) (size 0.975 1.4) (layers "B.Cu" "B.Paste" "B.Mask") (roundrect_rratio 0.25)
-      (net 199 "/sbbus1") (pinfunction "K") (pintype "passive"))
+      (net 199 "sbbus1") (pinfunction "K") (pintype "passive"))
     (pad "2" smd roundrect (at 0.9375 0) (size 0.975 1.4) (layers "B.Cu" "B.Paste" "B.Mask") (roundrect_rratio 0.25)
       (net 221 "VCC") (pinfunction "A") (pintype "passive"))
@@
       (stroke (width 0.1) (type solid)) (layer "B.Fab"))
     (pad "1" smd roundrect (at -0.9375 0 90) (size 0.975 1.4) (layers "B.Cu" "B.Paste" "B.Mask") (roundrect_rratio 0.25)
-      (net 200 "/sbbus2") (pinfunction "K") (pintype "passive"))
+      (net 200 "sbbus2") (pinfunction "K") (pintype "passive"))
     (pad "2" smd roundrect (at 0.9375 0 90) (size 0.975 1.4) (layers "B.Cu" "B.Paste" "B.Mask") (roundrect_rratio 0.25)
       (net 221 "VCC") (pinfunction "A") (pintype "passive"))
@@
       (stroke (width 0.1) (type solid)) (layer "B.Fab"))
     (pad "1" smd roundrect (at -0.9375 0 90) (size 0.975 1.4) (layers "B.Cu" "B.Paste" "B.Mask") (roundrect_rratio 0.25)
-      (net 201 "/scbus0") (pinfunction "K") (pintype "passive"))
+      (net 201 "scbus0") (pinfunction "K") (pintype "passive"))
     (pad "2" smd roundrect (at 0.9375 0 90) (size 0.975 1.4) (layers "B.Cu" "B.Paste" "B.Mask") (roundrect_rratio 0.25)
       (net 221 "VCC") (pinfunction "A") (pintype "passive"))
@@
       (stroke (width 0.1) (type solid)) (layer "B.Fab"))
     (pad "1" smd roundrect (at -0.9375 0) (size 0.975 1.4) (layers "B.Cu" "B.Paste" "B.Mask") (roundrect_rratio 0.25)
-      (net 202 "/scbus1") (pinfunction "K") (pintype "passive"))
+      (net 202 "scbus1") (pinfunction "K") (pintype "passive"))
     (pad "2" smd roundrect (at 0.9375 0) (size 0.975 1.4) (layers "B.Cu" "B.Paste" "B.Mask") (roundrect_rratio 0.25)
       (net 221 "VCC") (pinfunction "A") (pintype "passive"))
@@
       (stroke (width 0.1) (type solid)) (layer "B.Fab"))
     (pad "1" smd roundrect (at -0.9375 0 90) (size 0.975 1.4) (layers "B.Cu" "B.Paste" "B.Mask") (roundrect_rratio 0.25)
-      (net 203 "/scbus2") (pinfunction "K") (pintype "passive"))
+      (net 203 "scbus2") (pinfunction "K") (pintype "passive"))
     (pad "2" smd roundrect (at 0.9375 0 90) (size 0.975 1.4) (layers "B.Cu" "B.Paste" "B.Mask") (roundrect_rratio 0.25)
       (net 221 "VCC") (pinfunction "A") (pintype "passive"))

Commit message: V6 and V7 PCB
Parts:
- moved REF** 13.6 mm to (51.1, 124.0)
Other:
- board text added: "DSKY LED Display V7 Riley Rainey 2025-03-17"
- board text removed: "DSKY LED Display V6 Riley Rainey 2024-12-24"
